Commit message: Generate config for ur with gripper, setup motion planning

File: workspace/src/ur_with_2f_85_description/urdf/ur_with_2f_85.urdf.xacro (robot description, xacro)
@@ -1,10 +1,81 @@
 <?xml version="1.0"?>
 <robot xmlns:xacro="http://wiki.ros.org/xacro" name="robotiq_gripper">
-    <xacro:include filename="$(find ur_simulation_gz)/urdf/ur_gz.urdf.xacro" />
+    <!-- UR5e -->
+    <!-- robot name parameter -->
+    <xacro:arg name="name" default="ur"/>
+    <!-- import main macro -->
+    <xacro:include filename="$(find ur_description)/urdf/ur_macro.xacro"/>
+    <xacro:include filename="$(find ur_simulation_gz)/urdf/ur_gz.ros2_control.xacro" />
+    <!-- possible 'ur_type' values: ur3, ur3e, ur5, ur5e, ur7e, ur10, ur10e, ur12e, ur16e, ur15, ur20, ur30 -->
+    <!-- the default value should raise an error in case this was called without defining the type -->
+    <!-- Note(Vince Reda): Changed default to ur5e -->
+    <xacro:arg name="ur_type" default="ur5e"/>
+    <!-- parameters -->
+    <xacro:arg name="tf_prefix" default="" />
+    <xacro:arg name="parent" default="world"/>
+    <xacro:arg name="joint_limit_params" default="$(find ur_description)/config/$(arg ur_type)/joint_limits.yaml"/>
+    <xacro:arg name="kinematics_params" default="$(find ur_description)/config/$(arg ur_type)/default_kinematics.yaml"/>
+    <xacro:arg name="physical_params" default="$(find ur_description)/config/$(arg ur_type)/physical_parameters.yaml"/>
+    <xacro:arg name="visual_params" default="$(find ur_description)/config/$(arg ur_type)/visual_parameters.yaml"/>
+    <xacro:arg name="transmission_hw_interface" default=""/>
+    <xacro:arg name="safety_limits" default="false"/>
+    <xacro:arg name="safety_pos_margin" default="0.15"/>
+    <xacro:arg name="safety_k_position" default="20"/>
+    <xacro:arg name="simulation_controllers" default="" />
+    <xacro:arg name="ros_namespace" default="" />
+    <link name="$(arg parent)"/>
+    <!-- <link name="ground_plane"> -->
+    <!--   <visual> -->
+    <!--     <origin rpy="0 0 0" xyz="0 0 0"/> -->
+    <!--     <geometry> -->
+    <!--       <box size="5 5 0"/> -->
+    <!--     </geometry> -->
+    <!--     <material name="ground_white"> -->
+    <!--       <color rgba="1 1 1 0.5"/> -->
+    <!--     </material> -->
+    <!--   </visual> -->
+    <!--   <collision> -->
+    <!--     <origin rpy="0 0 0" xyz="0 0 0"/> -->
+    <!--     <geometry> -->
+    <!--       <box size="5 5 0"/> -->
+    <!--     </geometry> -->
+    <!--   </collision> -->
+    <!-- </link> -->
+    <!-- arm -->
+    <xacro:ur_robot
+      name="$(arg name)"
+      tf_prefix="$(arg tf_prefix)"
+      parent="$(arg parent)"
+      joint_limits_parameters_file="$(arg joint_limit_params)"
+      kinematics_parameters_file="$(arg kinematics_params)"
+      physical_parameters_file="$(arg physical_params)"
+      visual_parameters_file="$(arg visual_params)"
+      safety_limits="$(arg safety_limits)"
+      safety_pos_margin="$(arg safety_pos_margin)"
+      safety_k_position="$(arg safety_k_position)"
+      force_abs_paths="true"
+      >
+      <origin xyz="0 0 0" rpy="0 0 0" />          <!-- position robot in the fixed frame -->
+    </xacro:ur_robot>
+    <gazebo>
+      <plugin filename="gz_ros2_control-system" name="gz_ros2_control::GazeboSimROS2ControlPlugin">
+        <parameters>$(arg simulation_controllers)</parameters>
+        <ros>
+          <namespace>$(arg ros_namespace)</namespace>
+        </ros>
+      </plugin>
+    </gazebo>
+    <!-- ros2 control instance -->
+    <xacro:ur_ros2_control
+      name="$(arg name)"
+      tf_prefix="$(arg tf_prefix)"
+      transmission_hw_interface="$(arg transmission_hw_interface)"
+    />
+    <!-- Gripper -->
     <xacro:include filename="$(find robotiq_description)/urdf/robotiq_2f_85_macro.urdf.xacro" />
     <xacro:robotiq_gripper
             name="RobotiqGripperHardwareInterface"
             prefix=""
-            parent="tool0"
+            parent="wrist_3_link"
             sim_gazebo="true"
             use_fake_hardware="true">

Commit message: Add finger and gripper frames to urdf

File: workspace/src/ur_with_2f_85_description/urdf/ur_with_2f_85.urdf.xacro (robot description, xacro)
@@ -82,3 +82,26 @@
         <origin xyz="0 0 0" rpy="0 0 0" />
     </xacro:robotiq_gripper>
+    <!-- Add finger tip frames -->
+    <xacro:macro name="add_finger_tip_frame" params="side">
+      <link name="${side}_finger_tip_link"/>
+      <joint name="${side}_finger_tip_joint" type="fixed">
+        <parent link="robotiq_85_${side}_finger_tip_link"/>
+        <child link="${side}_finger_tip_link"/>
+        <xacro:if value="${side == 'left'}">
+          <origin xyz="-0.025 0 0.03" rpy="0 0 0"/>
+        </xacro:if>
+        <xacro:if value="${side == 'right'}">
+          <origin xyz="0.025 0 0.03" rpy="0 0 0"/>
+        </xacro:if>,
+      </joint>
+    </xacro:macro>
+    <xacro:add_finger_tip_frame side="left"/>
+    <xacro:add_finger_tip_frame side="right"/>
+    <!-- Add gripper frame -->
+    <link name="gripper_link"/>
+    <joint name="gripper_joint" type="fixed">
+        <parent link="wrist_3_link"/>
+        <child link="gripper_link"/>
+        <origin xyz="0 0 0.14" rpy="0 0 0"/>
+    </joint>
 </robot>

Commit message: Restructure description and config, visualize gripper

File: workspace/src/ur_with_2f_85_description/urdf/ur_with_2f_85.urdf.xacro (robot description, xacro)
@@ -99,8 +99,8 @@
     <xacro:add_finger_tip_frame side="right"/>
     <!-- Add gripper frame -->
-    <link name="gripper_link"/>
+    <link name="grasp_link"/>
     <joint name="gripper_joint" type="fixed">
         <parent link="wrist_3_link"/>
-        <child link="gripper_link"/>
+        <child link="grasp_link"/>
         <origin xyz="0 0 0.14" rpy="0 0 0"/>
     </joint>

Commit message: Finally solved collision detection bug

File: workspace/src/ur_with_2f_85_description/urdf/ur_with_2f_85.urdf.xacro (robot description, xacro)
@@ -103,5 +103,5 @@
         <parent link="wrist_3_link"/>
         <child link="grasp_link"/>
-        <origin xyz="0 0 0.14" rpy="0 0 0"/>
+        <origin xyz="0 0 0.133.7" rpy="0 0 0"/>
     </joint>
 </robot>
